File: dell7212/kicad/bgpogo/bgpogo.kicad_sch (KiCad schematic)
At the start: 5 parts, among them J1 Conn_02x13_Odd_Even, J2 USB1135-15-9-L-B_REVA1, U1 AZ1117-5.0

Commit message: pogo sch maybe ready
Parts:
- added J3, J6: Conn_01x13, symbol Connector_Generic:Conn_01x13
- added J4: PJ-019, libs:CUI_PJ-019, symbol PJ-019:PJ-019
- added J5: Conn_01x03, symbol Connector_Generic:Conn_01x03
- added J7: Conn_01x09, symbol Connector_Generic:Conn_01x09
- J1: footprint (none) -> pogo1:dell 72xx pogo
Connections:
- net +5V: now also J7.1 (Pin_1)
- net 53: now also J7.3 (Pin_3)
- net 54: now also J7.2 (Pin_2)
- net 55: now also J7.9 (Pin_9)
- net 56: now also J7.8 (Pin_8)
- net 58: now also J7.7 (Pin_7)
- net 59: now also J7.6 (Pin_6)
- net GND: now also U1.1 (GND), J3.3 (Pin_3), J7.4 (Pin_4), J7.5 (Pin_5)
- net p1: now reaches J1.1 (Pin_1)
- net p1: now also J3.1 (Pin_1)
- net p3: now reaches J1.3 (Pin_3)
- net p3: now also J3.2 (Pin_2)
- net p7: now reaches J1.7 (Pin_7)
- net p7: now also J3.4 (Pin_4)
- net p9: now reaches J1.9 (Pin_9)
- net p9: now also J3.5 (Pin_5)
- new net: J4.1, J5.1 (Pin_1)
- new net: J4.2, J5.3 (Pin_3)
- new net: J4.3, J5.2 (Pin_2)
- new net p10: J6.5 (Pin_5)
- new net p11: J3.6 (Pin_6)
- new net p12: J6.6 (Pin_6)
- new net p13: J3.7 (Pin_7)
- new net p14: J6.7 (Pin_7)
- new net p15: J3.8 (Pin_8)
- new net p16: J6.8 (Pin_8)
- new net p17: J3.9 (Pin_9)
- new net p18: J6.9 (Pin_9)
- new net p19: J3.10 (Pin_10)
- new net p2: J6.1 (Pin_1)
- new net p20: J6.10 (Pin_10)
- new net p21: J3.11 (Pin_11)
- new net p22: J6.11 (Pin_11)
- new net p23: J3.12 (Pin_12)
- new net p24: J6.12 (Pin_12)
- new net p25: J3.13 (Pin_13)
- new net p26: J6.13 (Pin_13)
- new net p4: J6.2 (Pin_2)
- new net p6: J6.3 (Pin_3)
- new net p8: J6.4 (Pin_4)
Other:
- moved on the sheet: C1, C2, J2, U1

Commit message: pogo sch assign header footprints.
Parts:
- J5: footprint (none) -> Connector_PinHeader_2.54mm:PinHeader_1x03_P2.54mm_Vertical
- J6: footprint (none) -> Connector_PinHeader_2.54mm:PinHeader_1x13_P2.54mm_Vertical
- J7: footprint (none) -> Connector_PinHeader_2.54mm:PinHeader_1x09_P2.54mm_Vertical
Changed lines of the file:
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@@
 			)
 		)
-		(property "Footprint" ""
+		(property "Footprint" "Connector_PinHeader_2.54mm:PinHeader_1x09_P2.54mm_Vertical"
 			(at 149.86 74.93 0)
 			(effects
@@
 			)
 		)
-		(property "Footprint" ""
+		(property "Footprint" "Connector_PinHeader_2.54mm:PinHeader_1x13_P2.54mm_Vertical"
 			(at 74.93 123.19 0)
 			(effects
@@
 			)
 		)
-		(property "Footprint" ""
+		(property "Footprint" "Connector_PinHeader_2.54mm:PinHeader_1x03_P2.54mm_Vertical"
 			(at 148.59 130.81 0)
 			(effects

Commit message: more nets.
Parts:
- J3: footprint (none) -> Connector_PinHeader_2.54mm:PinHeader_1x13_P2.54mm_Vertical
Connections:
- net p10 is gone; now on net 56: J6.5 (Pin_5)
- net p11 is gone; now on net GND: J3.6 (Pin_6)
- net p12 is gone; now on net GND: J6.6 (Pin_6)
- net p14 is gone; now on net 58: J6.7 (Pin_7)
- net p16 is gone; now on net 59: J6.8 (Pin_8)
- net p17 is gone; now on net GND: J3.9 (Pin_9)
- net p18 is gone; now on net GND: J6.9 (Pin_9)
- net p20 is gone; now on net 53: J6.10 (Pin_10)
- net p22 is gone; now on net 54: J6.11 (Pin_11)
- net p23 is gone; now on net +3.3V: J3.12 (Pin_12)
- net p24 is gone; now on net GND: J6.12 (Pin_12)
- net p25 is gone; now on net +8V: J3.13 (Pin_13)
- net p26 is gone; now on net +8V: J6.13 (Pin_13)
- net p6 is gone; now on net GND: J6.3 (Pin_3)
- net p8 is gone; now on net 55: J6.4 (Pin_4)
- net p13: now also J1.13 (Pin_13)
- net p15: now also J1.15 (Pin_15)
- net p19: now also J1.19 (Pin_19)
- net p2: now also J1.2 (Pin_2)
- net p21: now also J1.21 (Pin_21)
- net p4: now also J1.4 (Pin_4)

Commit message: board v.9
Parts:
- added H1, H2, H3, H4: MountingHole, MountingHole:MountingHole_2.5mm, symbol Mechanical:MountingHole
Connections:
- net +5V: now also J7.2 (Pin_2); no longer J7.1 (Pin_1)
- net 53: now also J7.6 (Pin_6); no longer J7.3 (Pin_3)
- net 54: now also J7.4 (Pin_4); no longer J7.2 (Pin_2)
- net 55: now also J7.1 (Pin_1); no longer J7.9 (Pin_9)
- net 56: now also J7.3 (Pin_3); no longer J7.8 (Pin_8)
- net 59: now also J7.9 (Pin_9); no longer J7.6 (Pin_6)
- net GND: now also J7.8 (Pin_8); no longer J7.4 (Pin_4)

Commit message: board v1.0 ordered
Parts:
- added J8: PJ-104H, PJ_104H:SAMESKY_PJ-104H, symbol PJ-104H:PJ-104H
- added J9: Conn_01x03, Connector_PinHeader_2.54mm:PinHeader_1x03_P2.54mm_Vertical, symbol Connector_Generic:Conn_01x03
Connections:
- new net: J8.1, J9.1 (Pin_1)
- new net: J8.3, J9.2 (Pin_2)
- new net: J8.2, J9.3 (Pin_3)
Changed lines of the file:
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@@
 	(wire
 		(pts
+			(xy 142.24 153.67) (xy 134.62 153.67)
+		)
+		(stroke
+			(width 0)
+			(type default)
+		)
+	)
+	(wire
+		(pts
 			(xy 114.3 92.71) (xy 111.76 92.71)
 		)
@@
 	(wire
 		(pts
+			(xy 142.24 156.21) (xy 134.62 156.21)
+		)
+		(stroke
+			(width 0)
+			(type default)
+		)
+	)
+	(wire
+		(pts
 			(xy 62.23 125.73) (xy 69.85 125.73)
 		)
@@
 	(wire
 		(pts
+			(xy 142.24 151.13) (xy 134.62 151.13)
+		)
+		(stroke
+			(width 0)
+			(type default)
+		)
+	)
+	(wire
+		(pts
 			(xy 41.91 71.12) (xy 48.26 71.12)
 		)
@@
 	)
 	(symbol
+		(lib_id "Connector_Generic:Conn_01x03")
+		(at 147.32 153.67 0)
+		(unit 1)
+		(exclude_from_sim no)
+		(in_bom yes)
+		(on_board yes)
+		(dnp no)
+		(fields_autoplaced yes)
+		(property "Reference" "J9"
+			(at 149.86 152.3999 0)
+			(effects
+				(font
+					(size 1.27 1.27)
+				)
+				(justify left)
+			)
+		)
+		(property "Value" "Conn_01x03"
+			(at 149.86 154.9399 0)
+			(effects
+				(font
+					(size 1.27 1.27)
+				)
+				(justify left)
+			)
+		)
+		(property "Footprint" "Connector_PinHeader_2.54mm:PinHeader_1x03_P2.54mm_Vertical"
+			(at 147.32 153.67 0)
+			(effects
+				(font
+					(size 1.27 1.27)
+				)
+				(hide yes)
+			)
+		)
+		(property "Datasheet" "~"
+			(at 147.32 153.67 0)
+			(effects
+				(font
+					(size 1.27 1.27)
+				)
+				(hide yes)
+			)
+		)
+		(property "Description" "Generic connector, single row, 01x03, script generated (kicad-library-utils/schlib/autogen/connector/)"
+			(at 147.32 153.67 0)
+			(effects
+				(font
+					(size 1.27 1.27)
+				)
+				(hide yes)
+			)
+		)
+		(pin "1"
+		)
+		(pin "2"
+		)
+		(pin "3"
+		)
+		(instances
+			(project "bgpogo"
+				(path "/32687b02-412d-4c2f-95b1-54c4396d397d"
+					(reference "J9")
+					(unit 1)
+				)
+			)
+		)
+	)
+	(symbol
 		(lib_id "Mechanical:MountingHole")
 		(at 158.75 54.61 0)
@@
 					(unit 1)
 				)
+			)
+		)
+	)
+	(symbol
+		(lib_id "PJ-104H:PJ-104H")
+		(at 124.46 153.67 0)
+		(unit 1)
+		(exclude_from_sim no)
+		(in_bom yes)
+		(on_board yes)
+		(dnp no)
+		(fields_autoplaced yes)
+		(property "Reference" "J8"
+			(at 124.46 144.78 0)
+			(effects
+				(font
+					(size 1.27 1.27)
+				)
+			)
+		)
+		(property "Value" "PJ-104H"
+			(at 124.46 147.32 0)
+			(effects
+				(font
+					(size 1.27 1.27)
+				)
+			)
+		)
+		(property "Footprint" "PJ_104H:SAMESKY_PJ-104H"
+			(at 124.46 153.67 0)
+			(effects
+				(font
+					(size 1.27 1.27)
+				)
+				(justify bottom)
+				(hide yes)
+			)
+		)
+		(property "Datasheet" ""
+			(at 124.46 153.67 0)
+			(effects
+				(font
+					(size 1.27 1.27)
+				)
+				(hide yes)
+			)
+		)
+		(property "Description" ""
+			(at 124.46 153.67 0)
+			(effects
+				(font
+					(size 1.27 1.27)
+				)
+				(hide yes)
+			)
+		)
+		(property "PARTREV" "1.0"
+			(at 124.46 153.67 0)
+			(effects
+				(font
+					(size 1.27 1.27)
+				)
+				(justify bottom)
+				(hide yes)
+			)
+		)
+		(property "STANDARD" "Manufacturer Recommendations"
+			(at 124.46 153.67 0)
+			(effects
+				(font
+					(size 1.27 1.27)
+				)
+				(justify bottom)
+				(hide yes)
+			)
+		)
+		(property "MAXIMUM_PACKAGE_HEIGHT" "7.8mm"
+			(at 124.46 153.67 0)
+			(effects
+				(font
+					(size 1.27 1.27)
+				)
+				(justify bottom)
+				(hide yes)
+			)
+		)
+		(property "MANUFACTURER" "Same Sky"
+			(at 124.46 153.67 0)
+			(effects
+				(font
+					(size 1.27 1.27)
+				)
+				(justify bottom)
+				(hide yes)
+			)
+		)
+		(pin "2"
+		)
+		(pin "3"
+		)
+		(pin "1"
+		)
+		(instances
+			(project ""
+				(path "/32687b02-412d-4c2f-95b1-54c4396d397d"
+					(reference "J8")
+					(unit 1)
+				)

Commit message: unground the groungs
Connections:
- net +8V: no longer J1.25 (Pin_25), J1.26 (Pin_26), J3.13 (Pin_13), J6.13 (Pin_13)
- net GND: no longer J1.11 (Pin_11), J1.12 (Pin_12), J1.17 (Pin_17), J1.18 (Pin_18), J1.24 (Pin_24), J1.5 (Pin_5), J1.6 (Pin_6), J3.3 (Pin_3), J3.6 (Pin_6), J3.9 (Pin_9), J6.12 (Pin_12), J6.3 (Pin_3), J6.6 (Pin_6), J6.9 (Pin_9)
- net +3.3V renamed p23
- new net p11: J1.11 (Pin_11), J3.6 (Pin_6)
- new net p12: J1.12 (Pin_12), J6.6 (Pin_6)
- new net p17: J1.17 (Pin_17), J3.9 (Pin_9)
- new net p18: J1.18 (Pin_18), J6.9 (Pin_9)
- new net p24: J1.24 (Pin_24), J6.12 (Pin_12)
- new net p25: J1.25 (Pin_25), J3.13 (Pin_13)
- new net p26: J1.26 (Pin_26), J6.13 (Pin_13)
- new net p5: J1.5 (Pin_5), J3.3 (Pin_3)
- new net p6: J1.6 (Pin_6), J6.3 (Pin_3)
